Commit message: [Fix] base_link and wheel joint

File: pir_description/urdf/pir_robot_frame.gazebo.xacro (robot description, xacro)
@@ -68,5 +68,5 @@
       <rightJoint>wheel_right_joint</rightJoint>
       <wheelSeparation>0.287</wheelSeparation>
-      <wheelDiameter>0.066</wheelDiameter>
+      <wheelDiameter>0.120</wheelDiameter>
       <wheelAcceleration>1</wheelAcceleration>
       <wheelTorque>10</wheelTorque>

File: pir_description/urdf/pir_robot_frame.urdf.xacro (robot description, xacro)
@@ -2,5 +2,5 @@
 <robot name="pir_robot_frame" xmlns:xacro="http://ros.org/wiki/xacro">
   <xacro:include filename="$(find pir_description)/urdf/common_properties.xacro"/>
-  <!--xacro:include filename="$(find pir_description)/urdf/pir_robot_frame.gazebo.xacro"/-->
+  <xacro:include filename="$(find pir_description)/urdf/pir_robot_frame.gazebo.xacro"/>
   <link name="base_footprint"/>
   <joint name="base_joint" type="fixed">
@@ -11,5 +11,5 @@
   <link name="base_link">
     <visual>
-      <origin xyz="0 0 0.0" rpy="0 0 0"/>
+      <origin xyz="0 0 0.04" rpy="0 0 0"/>
       <geometry>
         <!--box size="0.07 0.085 0.065"/-->
@@ -35,5 +35,5 @@
     <parent link="base_link"/>
     <child link="wheel_left_link"/>
-    <origin xyz="0.0 0.14 0.026" rpy="-1.57 0 0"/>
+    <origin xyz="0.0 0.14 0.056" rpy="-1.57 0 0"/>
     <axis xyz="0 0 1"/>
   </joint>
@@ -50,5 +50,5 @@
       <origin xyz="0 0 0" rpy="0 0 0"/>
       <geometry>
-        <cylinder length="0.018" radius="0.033"/>
+        <cylinder length="0.018" radius="0.06"/>
       </geometry>
     </collision>
@@ -64,5 +64,5 @@
     <parent link="base_link"/>
     <child link="wheel_right_link"/>
-    <origin xyz="0.0 -0.14 0.026" rpy="1.57 0 0"/>
+    <origin xyz="0.0 -0.14 0.056" rpy="1.57 0 0"/>
     <axis xyz="0 0 1"/>
   </joint>
@@ -79,5 +79,5 @@
       <origin xyz="0 0 0" rpy="0 0 0"/>
       <geometry>
-        <cylinder length="0.018" radius="0.033"/>
+        <cylinder length="0.018" radius="0.06"/>
       </geometry>
     </collision>

Commit message: [Edit] wheel color

File: pir_description/urdf/pir_robot_frame.gazebo.xacro (robot description, xacro)
@@ -15,5 +15,5 @@
     <maxVel>0.1</maxVel>
     <fdir1>1 0 0</fdir1>
-    <material>Gazebo/FlatBlack</material>
+    <material>Gazebo/LightGrey</material>
   </gazebo>
   <gazebo reference="wheel_right_link">
@@ -25,23 +25,5 @@
     <maxVel>0.1</maxVel>
     <fdir1>1 0 0</fdir1>
-    <material>Gazebo/FlatBlack</material>
-  </gazebo>
-  <gazebo reference="caster_back_right_link">
-    <mu1>0.1</mu1>
-    <mu2>0.1</mu2>
-    <kp>1000000.0</kp>
-    <kd>100.0</kd>
-    <minDepth>0.001</minDepth>
-    <maxVel>1.0</maxVel>
-    <material>Gazebo/FlatBlack</material>
-  </gazebo>
-  <gazebo reference="caster_back_left_link">
-    <mu1>0.1</mu1>
-    <mu2>0.1</mu2>
-    <kp>1000000.0</kp>
-    <kd>100.0</kd>
-    <minDepth>0.001</minDepth>
-    <maxVel>1.0</maxVel>
-    <material>Gazebo/FlatBlack</material>
+    <material>Gazebo/LightGrey</material>
   </gazebo>
   <gazebo reference="imu_link">

Commit message: [Fix] urdf model

File: pir_description/urdf/pir_robot_frame.gazebo.xacro (robot description, xacro)
@@ -33,4 +33,7 @@
     </sensor>
     <material>Gazebo/Grey</material>
+  </gazebo>
+  <gazebo reference="led_plate_link">
+    <material>Gazebo/Black</material>
   </gazebo>
   <gazebo>

File: pir_description/urdf/pir_robot_frame.urdf.xacro (robot description, xacro)
@@ -19,7 +19,7 @@
     </visual>
     <collision>
-      <origin xyz="0.0 0 0.095" rpy="0 0 0"/>
+      <origin xyz="0.0 0 0.085" rpy="0 0 0"/>
       <geometry>
-        <box size="0.266 0.266 0.184"/>
+        <box size="0.266 0.266 0.090"/>
       </geometry>
     </collision>
@@ -64,10 +64,10 @@
     <parent link="base_link"/>
     <child link="wheel_right_link"/>
-    <origin xyz="0.0 -0.14 0.056" rpy="1.57 0 3.14"/>
+    <origin xyz="0.0 -0.14 0.056" rpy="1.57 3.14 3.14"/>
     <axis xyz="0 0 1"/>
   </joint>
   <link name="wheel_right_link">
     <visual>
-      <origin xyz="0 0 0" rpy="1.57 0 0"/>
+      <origin xyz="0 0 0" rpy="1.57 3.14 0"/>
       <geometry>
         <!--box size="0.07 0.085 0.065"/-->
@@ -89,4 +89,44 @@
                izz="2.0712558e-05" />
       </inertial>
+  </link>
+  <joint name="caster_front_joint" type="fixed">
+    <parent link="base_link"/>
+    <child link="caster_front_link"/>
+    <origin xyz="-0.1 0 0.03" rpy="-1.57 0 0"/>
+  </joint>
+  <link name="caster_front_link">
+    <collision>
+      <origin xyz="0 0.015 0" rpy="0 0 0"/>
+      <geometry>
+        <box size="0.030 0.03 0.020"/>
+      </geometry>
+    </collision>
+    <inertial>
+      <origin xyz="0 0 0" />
+      <mass value="0.005" />
+      <inertia ixx="0.001" ixy="0.0" ixz="0.0"
+               iyy="0.001" iyz="0.0"
+               izz="0.001" />
+    </inertial>
+  </link>
+  <joint name="caster_rear_joint" type="fixed">
+    <parent link="base_link"/>
+    <child link="caster_rear_link"/>
+    <origin xyz="0.1 0 0.03" rpy="-1.57 0 0"/>
+  </joint>
+  <link name="caster_rear_link">
+    <collision>
+      <origin xyz="0 0.015 0" rpy="0 0 0"/>
+      <geometry>
+        <box size="0.030 0.03 0.020"/>
+      </geometry>
+    </collision>
+    <inertial>
+      <origin xyz="0 0 0" />
+      <mass value="0.005" />
+      <inertia ixx="0.001" ixy="0.0" ixz="0.0"
+               iyy="0.001" iyz="0.0"
+               izz="0.001" />
+    </inertial>
   </link>
   <joint name="imu_joint" type="fixed">
@@ -124,4 +164,18 @@
     </inertial>
   </link>
->
+  <joint name="led_plate_joint" type="continuous">
+    <parent link="base_link"/>
+    <child link="led_plate_link"/>
+    <origin xyz="0.0 0 0.26" rpy="0.0 0.0 0.0"/>
+    <axis xyz="0 0 1"/>
+  </joint>
+  <link name="led_plate_link">
+    <visual>
+      <origin xyz="0 0 0" rpy="0 0 0"/>
+      <geometry>
+        <box size="0.22 0.12 0.012"/>
+      </geometry>
+      <material name="dark"/>
+    </visual>
+  </link>
 </robot>

Commit message: [Delete] led_plate link

File: pir_description/urdf/pir_robot_frame.gazebo.xacro (robot description, xacro)
@@ -33,7 +33,4 @@
     </sensor>
     <material>Gazebo/Grey</material>
-  </gazebo>
-  <gazebo reference="led_plate_link">
-    <material>Gazebo/Black</material>
   </gazebo>
   <gazebo>

File: pir_description/urdf/pir_robot_frame.urdf.xacro (robot description, xacro)
@@ -164,18 +164,3 @@
     </inertial>
   </link>
-  <joint name="led_plate_joint" type="continuous">
-    <parent link="base_link"/>
-    <child link="led_plate_link"/>
-    <origin xyz="0.0 0 0.26" rpy="0.0 0.0 0.0"/>
-    <axis xyz="0 0 1"/>
-  </joint>
-  <link name="led_plate_link">
-    <visual>
-      <origin xyz="0 0 0" rpy="0 0 0"/>
-      <geometry>
-        <box size="0.22 0.12 0.012"/>
-      </geometry>
-      <material name="dark"/>
-    </visual>
-  </link>
 </robot>
