Commit message: [Fix] wheel coordination

File: pir_description/urdf/pir_robot_frame.urdf.xacro (robot description, xacro)
@@ -7,9 +7,9 @@
     <parent link="base_footprint"/>
     <child link="base_link" />
-    <origin xyz="0 0 0.04" rpy="0 0 0"/>
+    <origin xyz="0 0 0.010" rpy="0 0 0"/>
   </joint>
   <link name="base_link">
     <visual>
-      <origin xyz="0 0 0.04" rpy="0 0 0"/>
+      <origin xyz="0 0 0.03" rpy="0 0 0"/>
       <geometry>
         <!--box size="0.07 0.085 0.065"/-->
@@ -19,7 +19,7 @@
     </visual>
     <collision>
-      <origin xyz="-0.064 0 0.047" rpy="0 0 0"/>
+      <origin xyz="0.0 0 0.095" rpy="0 0 0"/>
       <geometry>
-        <box size="0.266 0.266 0.094"/>
+        <box size="0.266 0.266 0.184"/>
       </geometry>
     </collision>
@@ -64,5 +64,5 @@
     <parent link="base_link"/>
     <child link="wheel_right_link"/>
-    <origin xyz="0.0 -0.14 0.056" rpy="1.57 0 0"/>
+    <origin xyz="0.0 -0.14 0.056" rpy="1.57 0 3.14"/>
     <axis xyz="0 0 1"/>
   </joint>

Commit message: [Fix] base_scan joint

File: pir_description/urdf/pir_robot_frame.urdf.xacro (robot description, xacro)
@@ -99,5 +99,5 @@
     <parent link="base_link"/>
     <child link="base_scan"/>
-    <origin xyz="0 0 0.126" rpy="0 0 0"/>
+    <origin xyz="0 0 0.156" rpy="0 0 0"/>
   </joint>
   <link name="base_scan">

Commit message: [Fix] mass and collision

File: pir_description/urdf/pir_robot_frame.urdf.xacro (robot description, xacro)
@@ -25,5 +25,5 @@
     </collision>
     <inertial>
-      <origin xyz="0 0 0" rpy="0 0 0"/>
+      <origin xyz="0 0 0.03" rpy="0 0 0"/>
       <mass value="1.3729096e+00"/>
       <inertia ixx="8.7002718e-03" ixy="-4.7576583e-05" ixz="1.1160499e-04"
@@ -55,5 +55,5 @@
     <inertial>
       <origin xyz="0 0 0" />
-      <mass value="2.8498940e-02" />
+      <mass value="2.8498940e-01" />
       <inertia ixx="1.1175580e-05" ixy="-4.2369783e-11" ixz="-5.9381719e-09"
                iyy="1.1192413e-05" iyz="-1.4400107e-11"
@@ -84,5 +84,5 @@
     <inertial>
       <origin xyz="0 0 0" />
-      <mass value="2.8498940e-02" />
+      <mass value="2.8498940e-01" />
       <inertia ixx="1.1175580e-05" ixy="-4.2369783e-11" ixz="-5.9381719e-09"
                iyy="1.1192413e-05" iyz="-1.4400107e-11"
@@ -99,5 +99,5 @@
       <origin xyz="0 0.015 0" rpy="0 0 0"/>
       <geometry>
-        <box size="0.030 0.03 0.020"/>
+        <box size="0.030 0.035 0.020"/>
       </geometry>
     </collision>
@@ -119,5 +119,5 @@
       <origin xyz="0 0.015 0" rpy="0 0 0"/>
       <geometry>
-        <box size="0.030 0.03 0.020"/>
+        <box size="0.030 0.035 0.020"/>
       </geometry>
     </collision>
